Commit message: Refactored launch files and updated config parameters for improved SLAM implementation

File: src/my_slam_pkg/urdf/car.urdf.xacro (robot description, xacro)
@@ -1,11 +1,11 @@
 <?xml version="1.0"?>
-<robot name="my_autonomous_car" xmlns:xacro="http://www.ros.org/wiki/xacro">
+<robot name="my_slam_pkg" xmlns:xacro="http://www.ros.org/wiki/xacro">
   <!-- Robot Configuration -->
-  <link name="base_footprint"/>
-  <joint name="base_joint" type="fixed">
+<link name="base_footprint"/>
+<joint name="base_joint" type="fixed">
     <parent link="base_footprint"/>
     <child link="base_link"/>
     <origin xyz="0 0 0.1" rpy="0 0 0"/>
-  </joint>
+</joint>
   <!-- Colors -->
   <material name="black">
@@ -210,10 +210,10 @@
       <pose>0 0 0 0 0 0</pose>
       <visualize>true</visualize>
-      <update_rate>10</update_rate>
+      <update_rate>20</update_rate>
       <ray>
         <scan>
           <horizontal>
-            <samples>360</samples>
-            <resolution>1</resolution>
+            <samples>720</samples>
+            <resolution>0.5</resolution>
             <min_angle>-3.14159</min_angle>
             <max_angle>3.14159</max_angle>
@@ -221,6 +221,6 @@
         </scan>
         <range>
-          <min>0.3</min>
-          <max>10.0</max>
+          <min>0.15</min>
+          <max>12.0</max>
           <resolution>0.01</resolution>
         </range>
@@ -243,7 +243,4 @@
     <mu1>0.8</mu1>
     <mu2>0.8</mu2>
-    <kp>100000000.0</kp>
-    <kd>1.0</kd>
-    <fdir1>1 0 0</fdir1>
 </gazebo>
 <gazebo reference="front_right_wheel">
@@ -251,7 +248,4 @@
     <mu1>0.8</mu1>
     <mu2>0.8</mu2>
-    <kp>100000000.0</kp>
-    <kd>1.0</kd>
-    <fdir1>1 0 0</fdir1>
 </gazebo>
 <gazebo reference="rear_left_wheel">
@@ -259,7 +253,4 @@
     <mu1>0.8</mu1>
     <mu2>0.8</mu2>
-    <kp>100000000.0</kp>
-    <kd>1.0</kd>
-    <fdir1>1 0 0</fdir1>
 </gazebo>
 <gazebo reference="rear_right_wheel">
@@ -267,7 +258,4 @@
     <mu1>0.8</mu1>
     <mu2>0.8</mu2>
-    <kp>100000000.0</kp>
-    <kd>1.0</kd>
-    <fdir1>1 0 0</fdir1>
 </gazebo>
   <gazebo reference="lidar_link">

Commit message: final software

File: src/my_slam_pkg/urdf/car.urdf.xacro (robot description, xacro)
@@ -2,10 +2,10 @@
 <robot name="my_slam_pkg" xmlns:xacro="http://www.ros.org/wiki/xacro">
   <!-- Robot Configuration -->
-<link name="base_footprint"/>
-<joint name="base_joint" type="fixed">
+  <link name="base_footprint"/>
+  <joint name="base_joint" type="fixed">
     <parent link="base_footprint"/>
     <child link="base_link"/>
     <origin xyz="0 0 0.1" rpy="0 0 0"/>
-</joint>
+  </joint>
   <!-- Colors -->
   <material name="black">
@@ -30,4 +30,5 @@
     <inertial>
       <mass value="5.0"/>
+      <origin xyz="0 0 0" rpy="0 0 0"/>
       <inertia ixx="0.1" ixy="0" ixz="0" iyy="0.1" iyz="0" izz="0.1"/>
     </inertial>
@@ -48,14 +49,15 @@
     <inertial>
       <mass value="0.5"/>
-      <inertia ixx="0.001" ixy="0" ixz="0" iyy="0.001" iyz="0" izz="0.001"/>
-    </inertial>
-  </link>
- <joint name="front_left_wheel_joint" type="continuous">
+      <origin xyz="0 0 0" rpy="0 0 0"/>
+      <inertia ixx="0.001" ixy="0" ixz="0" iyy="0.001" iyz="0" izz="0.001"/>
+    </inertial>
+  </link>
+  <joint name="front_left_wheel_joint" type="continuous">
     <parent link="base_link"/>
     <child link="front_left_wheel"/>
     <origin xyz="0.15 0.17 -0.05" rpy="-1.5708 0 0"/>
     <axis xyz="0 0 1"/>
-    <dynamics damping="0.0" friction="0.0"/>
-</joint>
+    <dynamics damping="0.05" friction="0.05"/>
+  </joint>
   <!-- Front Right Wheel -->
   <link name="front_right_wheel">
@@ -73,14 +75,15 @@
     <inertial>
       <mass value="0.5"/>
-      <inertia ixx="0.001" ixy="0" ixz="0" iyy="0.001" iyz="0" izz="0.001"/>
-    </inertial>
-  </link>
-<joint name="front_right_wheel_joint" type="continuous">
+      <origin xyz="0 0 0" rpy="0 0 0"/>
+      <inertia ixx="0.001" ixy="0" ixz="0" iyy="0.001" iyz="0" izz="0.001"/>
+    </inertial>
+  </link>
+  <joint name="front_right_wheel_joint" type="continuous">
     <parent link="base_link"/>
     <child link="front_right_wheel"/>
     <origin xyz="0.15 -0.17 -0.05" rpy="-1.5708 0 0"/>
     <axis xyz="0 0 1"/>
-    <dynamics damping="0.0" friction="0.0"/>
-</joint>
+    <dynamics damping="0.05" friction="0.05"/>
+  </joint>
   <!-- Rear Left Wheel -->
   <link name="rear_left_wheel">
@@ -98,14 +101,15 @@
     <inertial>
       <mass value="0.5"/>
-      <inertia ixx="0.001" ixy="0" ixz="0" iyy="0.001" iyz="0" izz="0.001"/>
-    </inertial>
-  </link>
- <joint name="rear_left_wheel_joint" type="continuous">
+      <origin xyz="0 0 0" rpy="0 0 0"/>
+      <inertia ixx="0.001" ixy="0" ixz="0" iyy="0.001" iyz="0" izz="0.001"/>
+    </inertial>
+  </link>
+  <joint name="rear_left_wheel_joint" type="continuous">
     <parent link="base_link"/>
     <child link="rear_left_wheel"/>
     <origin xyz="-0.15 0.17 -0.05" rpy="-1.5708 0 0"/>
     <axis xyz="0 0 1"/>
-    <dynamics damping="0.0" friction="0.0"/>
-</joint>
+    <dynamics damping="0.05" friction="0.05"/>
+  </joint>
   <!-- Rear Right Wheel -->
   <link name="rear_right_wheel">
@@ -123,14 +127,15 @@
     <inertial>
       <mass value="0.5"/>
-      <inertia ixx="0.001" ixy="0" ixz="0" iyy="0.001" iyz="0" izz="0.001"/>
-    </inertial>
-  </link>
-<joint name="rear_right_wheel_joint" type="continuous">
+      <origin xyz="0 0 0" rpy="0 0 0"/>
+      <inertia ixx="0.001" ixy="0" ixz="0" iyy="0.001" iyz="0" izz="0.001"/>
+    </inertial>
+  </link>
+  <joint name="rear_right_wheel_joint" type="continuous">
     <parent link="base_link"/>
     <child link="rear_right_wheel"/>
     <origin xyz="-0.15 -0.17 -0.05" rpy="-1.5708 0 0"/>
     <axis xyz="0 0 1"/>
-    <dynamics damping="0.0" friction="0.0"/>
-</joint>
+    <dynamics damping="0.05" friction="0.05"/>
+  </joint>
   <!-- LiDAR Link -->
   <link name="lidar_link">
@@ -148,4 +153,5 @@
     <inertial>
       <mass value="0.1"/>
+      <origin xyz="0 0 0" rpy="0 0 0"/>
       <inertia ixx="0.001" ixy="0" ixz="0" iyy="0.001" iyz="0" izz="0.001"/>
     </inertial>
@@ -199,5 +205,5 @@
   </ros2_control>
   <!-- Gazebo ROS2 Control Plugin -->
- <gazebo>
+  <gazebo>
     <plugin name="gazebo_ros2_control" filename="libgazebo_ros2_control.so">
       <parameters>$(find my_slam_pkg)/config/controllers.yaml</parameters>
@@ -205,5 +211,5 @@
     </plugin>
   </gazebo>
-  <!-- LiDAR Sensor Configuration -->
+  <!-- LiDAR Sensor Configuration - Improved configuration -->
   <gazebo reference="lidar_link">
     <sensor type="ray" name="lidar">
@@ -225,7 +231,13 @@
           <resolution>0.01</resolution>
         </range>
+        <noise>
+          <type>gaussian</type>
+          <mean>0.0</mean>
+          <stddev>0.01</stddev>
+        </noise>
       </ray>
       <plugin name="laser_controller" filename="libgazebo_ros_ray_sensor.so">
         <ros>
+          <namespace>/</namespace>
           <remapping>~/out:=scan</remapping>
         </ros>
@@ -239,24 +251,36 @@
     <material>Gazebo/Blue</material>
   </gazebo>
-<gazebo reference="front_left_wheel">
-    <material>Gazebo/Black</material>
-    <mu1>0.8</mu1>
-    <mu2>0.8</mu2>
-</gazebo>
-<gazebo reference="front_right_wheel">
-    <material>Gazebo/Black</material>
-    <mu1>0.8</mu1>
-    <mu2>0.8</mu2>
-</gazebo>
-<gazebo reference="rear_left_wheel">
-    <material>Gazebo/Black</material>
-    <mu1>0.8</mu1>
-    <mu2>0.8</mu2>
-</gazebo>
-<gazebo reference="rear_right_wheel">
-    <material>Gazebo/Black</material>
-    <mu1>0.8</mu1>
-    <mu2>0.8</mu2>
-</gazebo>
+  <gazebo reference="front_left_wheel">
+    <material>Gazebo/Black</material>
+    <mu1>0.8</mu1>
+    <mu2>0.8</mu2>
+    <kp>500000.0</kp>
+    <kd>10.0</kd>
+    <fdir1>1 0 0</fdir1>
+  </gazebo>
+  <gazebo reference="front_right_wheel">
+    <material>Gazebo/Black</material>
+    <mu1>0.8</mu1>
+    <mu2>0.8</mu2>
+    <kp>500000.0</kp>
+    <kd>10.0</kd>
+    <fdir1>1 0 0</fdir1>
+  </gazebo>
+  <gazebo reference="rear_left_wheel">
+    <material>Gazebo/Black</material>
+    <mu1>0.8</mu1>
+    <mu2>0.8</mu2>
+    <kp>500000.0</kp>
+    <kd>10.0</kd>
+    <fdir1>1 0 0</fdir1>
+  </gazebo>
+  <gazebo reference="rear_right_wheel">
+    <material>Gazebo/Black</material>
+    <mu1>0.8</mu1>
+    <mu2>0.8</mu2>
+    <kp>500000.0</kp>
+    <kd>10.0</kd>
+    <fdir1>1 0 0</fdir1>
+  </gazebo>
   <gazebo reference="lidar_link">
     <material>Gazebo/Black</material>

Commit message: last soft

File: src/my_slam_pkg/urdf/car.urdf.xacro (robot description, xacro)
@@ -1,4 +1,6 @@
 <?xml version="1.0"?>
 <robot name="my_slam_pkg" xmlns:xacro="http://www.ros.org/wiki/xacro">
+  <!-- Arguments -->
+  <xacro:arg name="use_fake_hardware" default="false"/>
   <!-- Robot Configuration -->
   <link name="base_footprint"/>
@@ -162,5 +164,7 @@
     <origin xyz="0 0 0.1" rpy="0 0 0"/>
   </joint>
-  <!-- ROS2 Control Configuration -->
+ <!-- ROS2 Control Configuration -->
+<xacro:if value="$(arg use_fake_hardware)">
+  <!-- Gazebo simulated control -->
   <ros2_control name="car_control" type="system">
     <hardware>
@@ -204,11 +208,68 @@
     </joint>
   </ros2_control>
+</xacro:if>
+<xacro:unless value="$(arg use_fake_hardware)">
+  <!-- ESP32 hardware control -->
+  <ros2_control name="esp32_motor_controller" type="system">
+    <hardware>
+      <plugin>my_slam_pkg/ESP32HardwareInterface</plugin>
+      <param name="wheel_radius">0.05</param>
+      <param name="wheel_separation">0.34</param>
+      <param name="cmd_vel_topic">/cmd_vel</param>
+      <param name="joint_states_topic">/joint_states</param>
+    </hardware>
+    <!-- Front Left Wheel -->
+    <joint name="front_left_wheel_joint">
+      <command_interface name="velocity">
+        <param name="min">-10</param>
+        <param name="max">10</param>
+      </command_interface>
+      <state_interface name="position"/>
+      <state_interface name="velocity"/>
+    </joint>
+    <!-- Front Right Wheel -->
+    <joint name="front_right_wheel_joint">
+      <command_interface name="velocity">
+        <param name="min">-10</param>
+        <param name="max">10</param>
+      </command_interface>
+      <state_interface name="position"/>
+      <state_interface name="velocity"/>
+    </joint>
+    <!-- Rear Left Wheel -->
+    <joint name="rear_left_wheel_joint">
+      <command_interface name="velocity">
+        <param name="min">-10</param>
+        <param name="max">10</param>
+      </command_interface>
+      <state_interface name="position"/>
+      <state_interface name="velocity"/>
+    </joint>
+    <!-- Rear Right Wheel -->
+    <joint name="rear_right_wheel_joint">
+      <command_interface name="velocity">
+        <param name="min">-10</param>
+        <param name="max">10</param>
+      </command_interface>
+      <state_interface name="position"/>
+      <state_interface name="velocity"/>
+    </joint>
+  </ros2_control>
+</xacro:unless>
   <!-- Gazebo ROS2 Control Plugin -->
   <gazebo>
+  <xacro:if value="$(arg use_fake_hardware)">
     <plugin name="gazebo_ros2_control" filename="libgazebo_ros2_control.so">
       <parameters>$(find my_slam_pkg)/config/controllers.yaml</parameters>
       <robot_sim_type>gazebo_ros2_control/GazeboSystem</robot_sim_type>
     </plugin>
-  </gazebo>
+  </xacro:if>
+  <xacro:unless value="$(arg use_fake_hardware)">
+    <plugin name="gazebo_ros2_control" filename="libgazebo_ros2_control.so">
+      <parameters>$(find my_slam_pkg)/config/hardware_controllers.yaml</parameters>
+      <robot_sim_type>my_slam_pkg/ESP32HardwareInterface</robot_sim_type>
+    </plugin>
+  </xacro:unless>
+</gazebo>
   <!-- LiDAR Sensor Configuration - Improved configuration -->
   <gazebo reference="lidar_link">
