Commit message: ekf added

File: src/my_slam_pkg/urdf/esp32_real_robot.urdf.xacro (robot description, xacro)
@@ -1,4 +1,4 @@
 <?xml version="1.0"?>
-<robot name="esp32_robot" xmlns:xacro="http://www.ros.org/wiki/xacro">
+<robot name="esp32_complete_robot" xmlns:xacro="http://www.ros.org/wiki/xacro">
   <!-- Arguments -->
   <xacro:arg name="use_fake_hardware" default="false"/>
@@ -31,4 +31,7 @@
   <material name="green">
     <color rgba="0.0 0.8 0.0 1.0"/>
+  </material>
+  <material name="yellow">
+    <color rgba="1.0 1.0 0.0 1.0"/>
   </material>
   <!-- Base Link -->
@@ -127,123 +130,99 @@
     </inertial>
   </link>
-  <!-- IMU mounting joint - adjust position based on your mounting -->
+  <!-- IMU mounting joint -->
   <joint name="imu_joint" type="fixed">
     <parent link="base_link"/>
     <child link="imu_link"/>
-    <!-- Position: 5cm above base_link center, adjust X/Y based on your actual mounting -->
     <origin xyz="0.0 0.0 0.08" rpy="0 0 0"/>
   </joint>
+  <!-- ESP32 Controller Board Link -->
+  <link name="esp32_link">
+    <visual>
+      <geometry>
+        <box size="0.06 0.03 0.01"/>
+      </geometry>
+      <material name="yellow"/>
+    </visual>
+    <collision>
+      <geometry>
+        <box size="0.06 0.03 0.01"/>
+      </geometry>
+    </collision>
+    <inertial>
+      <mass value="0.05"/>
+      <origin xyz="0 0 0" rpy="0 0 0"/>
+      <inertia ixx="0.0001" ixy="0" ixz="0" iyy="0.0001" iyz="0" izz="0.0001"/>
+    </inertial>
+  </link>
+  <joint name="esp32_joint" type="fixed">
+    <parent link="base_link"/>
+    <child link="esp32_link"/>
+    <origin xyz="-0.1 0.0 0.06" rpy="0 0 0"/>
+  </joint>
   <!-- ROS2 Control Configuration -->
-  <xacro:if value="$(arg use_fake_hardware)">
-    <!-- Gazebo simulated control -->
-    <ros2_control name="car_control" type="system">
-      <hardware>
-        <plugin>gazebo_ros2_control/GazeboSystem</plugin>
-      </hardware>
-      <!-- Front Left Wheel -->
-      <joint name="front_left_wheel_joint">
-        <command_interface name="velocity">
-          <param name="min">-10</param>
-          <param name="max">10</param>
-        </command_interface>
-        <state_interface name="position"/>
-        <state_interface name="velocity"/>
-      </joint>
-      <!-- Front Right Wheel -->
-      <joint name="front_right_wheel_joint">
-        <command_interface name="velocity">
-          <param name="min">-10</param>
-          <param name="max">10</param>
-        </command_interface>
-        <state_interface name="position"/>
-        <state_interface name="velocity"/>
-      </joint>
-      <!-- Rear Left Wheel -->
-      <joint name="rear_left_wheel_joint">
-        <command_interface name="velocity">
-          <param name="min">-10</param>
-          <param name="max">10</param>
-        </command_interface>
-        <state_interface name="position"/>
-        <state_interface name="velocity"/>
-      </joint>
-      <!-- Rear Right Wheel -->
-      <joint name="rear_right_wheel_joint">
-        <command_interface name="velocity">
-          <param name="min">-10</param>
-          <param name="max">10</param>
-        </command_interface>
-        <state_interface name="position"/>
-        <state_interface name="velocity"/>
-      </joint>
-    </ros2_control>
-  </xacro:if>
-  <xacro:unless value="$(arg use_fake_hardware)">
-    <!-- ESP32 hardware control -->
-    <ros2_control name="esp32_motor_controller" type="system">
-      <hardware>
-        <plugin>my_slam_pkg/ESP32HardwareInterface</plugin>
-        <param name="wheel_radius">0.05</param>
-        <param name="wheel_separation">0.34</param>
-        <param name="cmd_vel_topic">/cmd_vel</param>
-        <param name="joint_states_topic">/joint_states</param>
-        <param name="use_sim_hardware">false</param>
-      </hardware>
-      <!-- Front Left Wheel -->
-      <joint name="front_left_wheel_joint">
-        <command_interface name="velocity">
-          <param name="min">-10</param>
-          <param name="max">10</param>
-        </command_interface>
-        <state_interface name="position"/>
-        <state_interface name="velocity"/>
-        <state_interface name="effort"/>
-      </joint>
-      <!-- Front Right Wheel -->
-      <joint name="front_right_wheel_joint">
-        <command_interface name="velocity">
-          <param name="min">-10</param>
-          <param name="max">10</param>
-        </command_interface>
-        <state_interface name="position"/>
-        <state_interface name="velocity"/>
-        <state_interface name="effort"/>
-      </joint>
-      <!-- Rear Left Wheel -->
-      <joint name="rear_left_wheel_joint">
-        <command_interface name="velocity">
-          <param name="min">-10</param>
-          <param name="max">10</param>
-        </command_interface>
-        <state_interface name="position"/>
-        <state_interface name="velocity"/>
-        <state_interface name="effort"/>
-      </joint>
-      <!-- Rear Right Wheel -->
-      <joint name="rear_right_wheel_joint">
-        <command_interface name="velocity">
-          <param name="min">-10</param>
-          <param name="max">10</param>
-        </command_interface>
-        <state_interface name="position"/>
-        <state_interface name="velocity"/>
-        <state_interface name="effort"/>
-      </joint>
-    </ros2_control>
-  </xacro:unless>
+  <ros2_control name="esp32_hardware_system" type="system">
+    <hardware>
+      <plugin>my_slam_pkg/ESP32HardwareInterface</plugin>
+      <param name="use_sim_hardware">$(arg use_fake_hardware)</param>
+      <param name="wheel_radius">0.05</param>
+      <param name="wheel_separation">0.34</param>
+      <param name="cmd_vel_topic">/cmd_vel</param>
+      <param name="joint_states_topic">/joint_states</param>
+      <param name="odom_topic">/odom</param>
+      <param name="use_stamped_vel">false</param>
+    </hardware>
+    <!-- Front Left Wheel -->
+    <joint name="front_left_wheel_joint">
+      <command_interface name="velocity">
+        <param name="min">-10</param>
+        <param name="max">10</param>
+      </command_interface>
+      <state_interface name="position"/>
+      <state_interface name="velocity"/>
+      <state_interface name="effort"/>
+    </joint>
+    <!-- Front Right Wheel -->
+    <joint name="front_right_wheel_joint">
+      <command_interface name="velocity">
+        <param name="min">-10</param>
+        <param name="max">10</param>
+      </command_interface>
+      <state_interface name="position"/>
+      <state_interface name="velocity"/>
+      <state_interface name="effort"/>
+    </joint>
+    <!-- Rear Left Wheel -->
+    <joint name="rear_left_wheel_joint">
+      <command_interface name="velocity">
+        <param name="min">-10</param>
+        <param name="max">10</param>
+      </command_interface>
+      <state_interface name="position"/>
+      <state_interface name="velocity"/>
+      <state_interface name="effort"/>
+    </joint>
+    <!-- Rear Right Wheel -->
+    <joint name="rear_right_wheel_joint">
+      <command_interface name="velocity">
+        <param name="min">-10</param>
+        <param name="max">10</param>
+      </command_interface>
+      <state_interface name="position"/>
+      <state_interface name="velocity"/>
+      <state_interface name="effort"/>
+    </joint>
+  </ros2_control>
   <!-- Gazebo ROS2 Control Plugin -->
   <gazebo>
-    <xacro:if value="$(arg use_fake_hardware)">
-      <plugin name="gazebo_ros2_control" filename="libgazebo_ros2_control.so">
+    <plugin name="gazebo_ros2_control" filename="libgazebo_ros2_control.so">
+      <xacro:if value="$(arg use_fake_hardware)">
         <parameters>$(find my_slam_pkg)/config/controllers.yaml</parameters>
         <robot_sim_type>gazebo_ros2_control/GazeboSystem</robot_sim_type>
-      </plugin>
-    </xacro:if>
-    <xacro:unless value="$(arg use_fake_hardware)">
-      <plugin name="gazebo_ros2_control" filename="libgazebo_ros2_control.so">
-        <parameters>$(find my_slam_pkg)/config/hardware_controllers.yaml</parameters>
+      </xacro:if>
+      <xacro:unless value="$(arg use_fake_hardware)">
+        <parameters>$(find my_slam_pkg)/config/esp32_controllers.yaml</parameters>
         <robot_sim_type>my_slam_pkg/ESP32HardwareInterface</robot_sim_type>
-      </plugin>
-    </xacro:unless>
+      </xacro:unless>
+    </plugin>
   </gazebo>
   <!-- LiDAR Sensor Configuration -->
@@ -294,5 +273,5 @@
       </plugin>
       <always_on>true</always_on>
-      <update_rate>50</update_rate>
+      <update_rate>100</update_rate>
       <visualize>true</visualize>
       <imu>
@@ -394,3 +373,6 @@
     <material>Gazebo/Green</material>
   </gazebo>
+  <gazebo reference="esp32_link">
+    <material>Gazebo/Yellow</material>
+  </gazebo>
 </robot>
